File: Regulators.sch (KiCad schematic (older format))
At the start: 65 parts, among them J900 BARREL_JACK, SW5 SWITCH_INV, U6 AME8805, U7 ZT1412

Commit message: Updates in progress
Parts:
- added Q1, Q2: PNP, ~, symbol PNP
- added R151, R154: 0R, ~, symbol R
Connections:
- net labels added: DDR_V_CTRL, PWR_2V6_A, PWR_2V6_MAIN, PWR_A__2V6_MAIN, PWR_B__1V2_A, PWR_B__1V2_MAIN
- net labels removed: PWR_1V2_A
- wire segments 123 -> 138
Other:
- moved on the sheet: C105, C107, C108, C115, C117, C152, C155, C217, C236, C237, C242, C243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

Commit message: update
Parts:
- added R183, R213, R214: R, ~, symbol R
Connections:
- net labels added: PWR_3V3_B, PWR_3V3_C, PWR_3V3_D
- wire segments 138 -> 209
Other:
- note added: "POWER RAILS"
- moved on the sheet: C105, C107, C108, C115, C117, C151, C152, C155, C170, C217, C236, C237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

Commit message: Final commit
Parts:
- removed C152: C, ~, symbol C
- added C100, C101, C141, C144, C145, C148, C149, C174: C, ~, symbol C-RESCUE-Regulators
- C105, C107, C108, C109, C110, C115, C117, C155, C217, C226, C236, C237, C242, C243, C250, C265, C331, C416, C612, C68, C69, C75, C76, C77, C78, C99: symbol C -> C-RESCUE-Regulators
- C151: value C -> 70pF; symbol C -> C-RESCUE-Regulators
- C170: value C -> 2uF; symbol C -> C-RESCUE-Regulators
- C414: symbol CP1 -> CP1-RESCUE-Regulators
- C415, C617: value C -> 100nF; symbol C -> C-RESCUE-Regulators
- C417: value C -> 200nF; symbol C -> C-RESCUE-Regulators
- C423: value C -> 25uF; symbol C -> C-RESCUE-Regulators
- C44: value C -> 10nF; symbol C -> C-RESCUE-Regulators
- C45: renamed from C?; value C -> 10nF; symbol C -> C-RESCUE-Regulators
- C618: renamed from C?; value C -> 100nF; symbol C -> C-RESCUE-Regulators
- D72: value DIODESCH -> SK23
- L3: value INDUCTOR_SMALL -> 75uH
- L5: value INDUCTOR_SMALL -> 24uH
- R1: renamed from R?; value R -> 0R; symbol R -> R-RESCUE-Regulators
- R129: value R -> 38.7K; symbol R -> R-RESCUE-Regulators
- R130: value R -> 1K; symbol R -> R-RESCUE-Regulators
- R136, R151, R152, R154, R155, R24, R74, R75, R913, R914: symbol R -> R-RESCUE-Regulators
- R183, R213, R214, R273: value R -> 0R; symbol R -> R-RESCUE-Regulators
- R25: renamed from R?; value R -> 75R; symbol R -> R-RESCUE-Regulators
- R270: value R -> 38K; symbol R -> R-RESCUE-Regulators
- R51: renamed from R?; value R -> 300K; symbol R -> R-RESCUE-Regulators
- R60: value R -> 1R; symbol R -> R-RESCUE-Regulators
- R680: renamed from R?; symbol R -> R-RESCUE-Regulators
- gave numbers to parts that had none: 2
Connections:
- net labels removed: +1.2V
- wire segments 209 -> 145
Other:
- note added: "DC Input"
- note added: "Decoupling Capacitors"
- note added: "Kandó Kálmán Villamosmérnöki kar"
- note added: "Készítette: Bán Zoltán"
- note added: "Power Rails"
- note added: "Regulators"
- note removed: "POWER RAILS"
- moved on the sheet: C109, C110, C226, C331, C415, C416, C423, C612, C617, C618, D72, J900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
