File: SoC_DDR.sch (KiCad schematic (older format))
At the start: 105 parts, among them J3 RJ45_UNSHIELDED, J4/A RJ45_UNSHIELDED, J4/B RJ45_UNSHIELDED, J4/C RJ45_UNSHIELDED, J4/D RJ45_UNSHIELDED

Commit message: Updates in progress
Connections:
- net labels added: DDR_V_CTRL, LED1_LAN1, LED1_LAN2, LED1_LAN3, LED1_LAN4, LED1_WAN, LED2_LAN1, LED2_LAN2, LED2_LAN3, LED2_LAN4, LED2_WAN, PWR_A__1V2_D, SPI_CLK, SPI_CS, SPI_MISO, SPI_MOSI, UART_RX, UART_TX, WPS_BTN
- wire segments 407 -> 425
- no-connect marks 0 -> 2
Other:
- moved on the sheet: C15, C19, C250, C27, C29, C32, C33, C34, C35, C36, C37, C38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

Commit message: update
Parts:
- added D2: LED_WAN, ~, symbol DUAL_LED
- added D4: LED_LAN1, ~, symbol DUAL_LED
- added D5: LED_LAN2, ~, symbol DUAL_LED
- added D6: LED_LAN3, ~, symbol DUAL_LED
- added D7: LED_LAN4, ~, symbol DUAL_LED
- added J1: CONN_7X2, symbol CONN_7X2
- added R148: R, ~, symbol R
- added R179, R180, R181, R182, R195, R196, R198, R200, R201, R202: 180R, ~, symbol R
- added U2: MX25L3206E, ~, symbol MX25L3206E
- gave numbers to parts that had none: 5
Connections:
- net GND: now also U4.34 (VSS), U4.48 (VSS), U4.66 (VSS), J1.10, J1.2 (P2), J1.4 (P4), J1.6 (P6), J1.8 (P8), U2.4 (GND); no longer C43.1
- net LED1_LAN1: now also D4.A1
- net LED1_LAN2: now also D5.A1
- net LED1_LAN3: now also D6.A1
- net LED1_LAN4: now also D7.A1
- net LED1_WAN: now also D2.A1
- net LED2_LAN1: now also D4.A2
- net LED2_LAN3: now also D6.A2
- net LED2_LAN4: now also D7.A2
- net LED2_WAN: now also D2.A2
- net PWR_3V3_A: now also R179.2, R180.2, R181.2, R182.2, R195.2, R196.2, R198.2, R200.2, R201.2, R202.2, U2.3 (WP), U2.7 (HOLD), U2.8 (VCC)
- net SPI_CLK: now also U2.6 (SCLK)
- net SPI_MISO: now also U2.2 (SO)
- net SPI_MOSI: now also U2.5 (SI)
- net PWR_2V6_A: now reaches U3.1 (VDD_DDR), U3.119 (VDD_DDR), U3.32 (VDD_DDR)
- net PWR_2V6_A: now also U4.1 (VDD), U4.12 (VSSQ), U4.15 (VDDQ), U4.18 (VDD), U4.3 (VDDQ), U4.33 (VDD), U4.52 (VSSQ), U4.55 (VDDQ), U4.58 (VSSQ), U4.6 (VSSQ), U4.61 (VDDQ), U4.64 (VSSQ), U4.9 (VDDQ)
- net VDD_2V5: now reaches U3.105 (AVDD25), U3.114 (VDD25), U3.45 (VDD25), U3.55 (VDD25), U3.65 (VDD25), U3.72 (VDD25), U3.83 (VDD25), U3.96 (VDD25)
- net VDD_2V5: now also J1.14
- net SYS_RST_OUT_L: now reaches U3.111 (SYS_RST_OUT_L)
- net TDO/GPIO7: now reaches U3.82 (GPIO7/TDO)
- net TDO/GPIO7: now also J1.5 (P5)
- net TCK: now reaches U3.85 (TCK)
- net TCK: now also J1.9
- net RST_L: now reaches U3.93 (RST_L)
- net LED2_LAN2 renamed LED2_LAN2/TDI
- net LED2_LAN2/TDI: now also D5.A2, J1.7 (P7)
- net SPI_CS renamed SPI_CS/GPIO2
- net SPI_CS/GPIO2: now also J1.3 (P3), U2.1 (CS)
- new net: D2.K1, R202.1
- new net: D2.K2, R200.1
- new net: D6.K1, R181.1
- new net: D6.K2, R198.1
- new net: D7.K1, R182.1
- new net: D7.K2, R201.1
- new net: D4.K1, R195.1
- new net: D4.K2, R179.1
- new net: D5.K1, R180.1
- new net: D5.K2, R196.1
- new net: J1.11, R148.2
- no-connect marks 2 -> 11
Other:
- note added: "NO PLACED"
- note added: "R14\n"
- note added: "R55"
- note added: "R56\n"
- note added: "R85"
- moved on the sheet: C15, C19, C250, C27, C29, C32, C33, C34, C35, C36, C37, C38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

Commit message: Final commit
Parts:
- added 100nF: C241, symbol C
- added D9: LED_WPS, symbol LED
- added JP1: CONN_01X04, symbol CONN_01X04
- added R149: 1R, ~, symbol R-RESCUE-SoC_DDR
- added R190: 0R, ~, symbol R-RESCUE-SoC_DDR
- added R191: 10K, ~, symbol R-RESCUE-SoC_DDR
- added R83: 2.4K, ~, symbol R-RESCUE-SoC_DDR
- added SW2: WPS_Button, symbol SW_PUSH
- added Y1: CRYSTAL_SMD, symbol CRYSTAL_SMD
- C15, C19, C250, C27, C29, C32, C33, C34, C35, C36, C37, C38, C39, C40, C41, C42, C43: symbol C -> C-RESCUE-SoC_DDR
- R10, R107, R108, R109, R110, R111, R112, R116, R12, R124, R125, R126, R127, R13, R131, R132, R133, R134, R135, R137, R138, R142, R143, R145, R15, R158, R159, R16, R160, R161, R162, R163, R164, R165, R166, R17, R179, R18, R180, R181, R182, R19, R195, R196, R198, R20, R200, R201, R202, R21, R22, R23, R25, R26, R30, R31, R32, R34, R35, R36, R37, R38, R39, R40, R41, R42, R43, R44, R45, R46, R47, R48, R49, R50, R9: symbol R -> R-RESCUE-SoC_DDR
- R100, R102, R106, R120, R121, R122, R127, R128, R141, R142, R157: value R -> 50R; symbol R -> R-RESCUE-SoC_DDR
- R148: value R -> 1k; symbol R -> R-RESCUE-SoC_DDR
Connections:
- net labels added: REFCLK
- wire segments 512 -> 546
- no-connect marks 11 -> 12
Other:
- note added: "Flash Memory"
- note added: "JATG Header"
- note added: "Kandó Kálmán Villamosmérnöki kar"
- note added: "Készítette: Bán Zoltán"
- note added: "Oscillator"
- note added: "Status Leds"
- note added: "UART Header"
- note added: "WPS Switch"
- moved on the sheet: J1, R100, R102, R106, R107, R108, R109, R110, R111, R112, R116, R120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
